Commit message: reee

File: src/crobot_description/description/ros2_control.xacro (robot description, xacro)
@@ -22,7 +22,4 @@
         <param name="sweeper_name">sweeper_joint</param>
         <param name="winch_name">winch_joint</param>
-        <joint name="flagdropper_joint">
-          <command_interface name="velocity"/>
-        </joint>
         <!-- TODO: Confirm parameters -->
         <param name="loop_rate">30.0</param>
@@ -81,4 +78,9 @@
       <state_interface   name="velocity"/>
     </joint>
+    <joint name="flagdropper_joint">
+      <command_interface name="position"/>
+      <state_interface name="position"/>
+      <!-- <state_interface name="velocity"/>  -->
+    </joint>
   </ros2_control>
   <xacro:if value="$(arg sim_mode)">

Commit message: the working comp code

File: src/crobot_description/description/ros2_control.xacro (robot description, xacro)
@@ -78,9 +78,9 @@
       <state_interface   name="velocity"/>
     </joint>
+<!--
     <joint name="flagdropper_joint">
       <command_interface name="position"/>
       <state_interface name="position"/>
-      <!-- <state_interface name="velocity"/>  -->
-    </joint>
+    </joint> -->
   </ros2_control>
   <xacro:if value="$(arg sim_mode)">
